File: aalto-1/aalto-1.sch (KiCad schematic (older format))
At the start: 0 parts

Commit message: added CC2500 to schematic
Parts:
- added IC?: CC2500-RTY1, QFN50P400X400X90-21N, symbol CC2500-RTY1:CC2500-RTY1
Changed lines of the file:
@@
+	1    0    0    -1
+$EndComp
+$Comp
+L CC2500-RTY1:CC2500-RTY1 IC?
+U 1 1 603BE95F
+P 5150 4000
+F 0 "IC?" H 6594 3696 50  0000 L CNN
+F 1 "CC2500-RTY1" H 6594 3605 50  0000 L CNN
+F 2 "QFN50P400X400X90-21N" H 6400 4500 50  0001 L CNN
+F 3 "" H 6400 4400 50  0001 L CNN
+F 4 "RF Transceiver" H 6400 4300 50  0001 L CNN "Description"
+F 5 "" H 6400 4200 50  0001 L CNN "Height"
+F 6 "Texas Instruments" H 6400 4100 50  0001 L CNN "Manufacturer_Name"
+F 7 "CC2500-RTY1" H 6400 4000 50  0001 L CNN "Manufacturer_Part_Number"
+F 8 "839-CC2500-RTY1" H 6400 3900 50  0001 L CNN "Mouser Part Number"
+F 9 "https://www.mouser.com/Search/Refine.aspx?Keyword=839-CC2500-RTY1" H 6400 3800 50  0001 L CNN "Mouser Price/Stock"
+F 10 "" H 6400 3700 50  0001 L CNN "Arrow Part Number"
+F 11 "" H 6400 3600 50  0001 L CNN "Arrow Price/Stock"
+	1    5150 4000
 	1    0    0    -1
 $EndComp

Commit message: Testing adding lib files
Parts:
- IC?: symbol CC2500-RTY1:CC2500-RTY1 -> aalto-1-rescue:CC2500-RTY1-CC2500-RTY1
Changed lines of the file:
@@
 $EndComp
 $Comp
-L CC2500-RTY1:CC2500-RTY1 IC?
+L aalto-1-rescue:CC2500-RTY1-CC2500-RTY1 IC?
 U 1 1 603BE95F
 P 5150 4000

Commit message: added MSP to schematic
Parts:
- added IC?: MSP430F2274IYFFR, BGA49C40P7X7_333X349X62, symbol MSP430F2274IYFFR:MSP430F2274IYFFR
Changed lines of the file:
@@
+	1    0    0    -1
+$EndComp
+$Comp
+L MSP430F2274IYFFR:MSP430F2274IYFFR IC?
+U 1 1 603BEFA5
+P 6800 850
+F 0 "IC?" H 8350 1115 50  0000 C CNN
+F 1 "MSP430F2274IYFFR" H 8350 1024 50  0000 C CNN
+F 2 "BGA49C40P7X7_333X349X62" H 9750 950 50  0001 L CNN
+F 3 "http://www.ti.com/lit/gpn/msp430f2274" H 9750 850 50  0001 L CNN
+F 4 "16-bit Ultra-Low-Power Microcontroller, 32KB Flash, 1K RAM" H 9750 750 50  0001 L CNN "Description"
+F 5 "0.625" H 9750 650 50  0001 L CNN "Height"
+F 6 "Texas Instruments" H 9750 550 50  0001 L CNN "Manufacturer_Name"
+F 7 "MSP430F2274IYFFR" H 9750 450 50  0001 L CNN "Manufacturer_Part_Number"
+F 8 "595-MSP430F2274IYFFR" H 9750 350 50  0001 L CNN "Mouser Part Number"
+F 9 "https://www.mouser.com/Search/Refine.aspx?Keyword=595-MSP430F2274IYFFR" H 9750 250 50  0001 L CNN "Mouser Price/Stock"
+F 10 "MSP430F2274IYFFR" H 9750 150 50  0001 L CNN "Arrow Part Number"
+F 11 "https://www.arrow.com/en/products/msp430f2274iyffr/texas-instruments" H 9750 50  50  0001 L CNN "Arrow Price/Stock"
+	1    6800 850
 	1    0    0    -1
 $EndComp

Commit message: added crystal
Parts:
- added Y?: ABM11W-26.0000MHZ-6-D1X-T3, ABM11W300000MHZ4B1UT3, symbol ABM11W-26.0000MHZ-6-D1X-T3:ABM11W-26.0000MHZ-6-D1X-T3
- IC?: symbol MSP430F2274IYFFR:MSP430F2274IYFFR -> aalto-1-rescue:MSP430F2274IYFFR-MSP430F2274IYFFR
Changed lines of the file:
@@
 $EndComp
 $Comp
-L MSP430F2274IYFFR:MSP430F2274IYFFR IC?
+L aalto-1-rescue:MSP430F2274IYFFR-MSP430F2274IYFFR IC?
 U 1 1 603BEFA5
 P 6800 850
@@
 	1    0    0    -1
 $EndComp
+$Comp
+L ABM11W-26.0000MHZ-6-D1X-T3:ABM11W-26.0000MHZ-6-D1X-T3 Y?
+U 1 1 603BF50A
+P 1950 2250
+F 0 "Y?" H 2750 2515 50  0000 C CNN
+F 1 "ABM11W-26.0000MHZ-6-D1X-T3" H 2750 2424 50  0000 C CNN
+F 2 "ABM11W300000MHZ4B1UT3" H 3400 2350 50  0001 L CNN
+F 3 "https://abracon.com/Resonators/ABM11W.pdf" H 3400 2250 50  0001 L CNN
+F 4 "Crystals 26MHz 6pF -40C +85C 10ppm" H 3400 2150 50  0001 L CNN "Description"
+F 5 "0" H 3400 2050 50  0001 L CNN "Height"
+F 6 "ABRACON" H 3400 1950 50  0001 L CNN "Manufacturer_Name"
+F 7 "ABM11W-26.0000MHZ-6-D1X-T3" H 3400 1850 50  0001 L CNN "Manufacturer_Part_Number"
+F 8 "815-11W26-6D1XT" H 3400 1750 50  0001 L CNN "Mouser Part Number"
+F 9 "https://www.mouser.co.uk/ProductDetail/ABRACON/ABM11W-260000MHZ-6-D1X-T3/?qs=5aG0NVq1C4z1GA6BiaLhDQ%3D%3D" H 3400 1650 50  0001 L CNN "Mouser Price/Stock"
+F 10 "" H 3400 1550 50  0001 L CNN "Arrow Part Number"
+F 11 "" H 3400 1450 50  0001 L CNN "Arrow Price/Stock"
+	1    1950 2250
+	1    0    0    -1
+$EndComp

Commit message: added power switch
Parts:
- added IC?: TPS2556DRBR, SON65P300X300X100-9N, symbol TPS2556DRBR:TPS2556DRBR
- Y?: symbol ABM11W-26.0000MHZ-6-D1X-T3:ABM11W-26.0000MHZ-6-D1X-T3 -> aalto-1-rescue:ABM11W-26.0000MHZ-6-D1X-T3-ABM11W-26.0000MHZ-6-D1X-T3
Changed lines of the file:
@@
 $EndComp
 $Comp
-L ABM11W-26.0000MHZ-6-D1X-T3:ABM11W-26.0000MHZ-6-D1X-T3 Y?
+L aalto-1-rescue:ABM11W-26.0000MHZ-6-D1X-T3-ABM11W-26.0000MHZ-6-D1X-T3 Y?
 U 1 1 603BF50A
 P 1950 2250
@@
 	1    0    0    -1
 $EndComp
+$Comp
+L TPS2556DRBR:TPS2556DRBR IC?
+U 1 1 603C13A8
+P 2000 4750
+F 0 "IC?" H 2600 5015 50  0000 C CNN
+F 1 "TPS2556DRBR" H 2600 4924 50  0000 C CNN
+F 2 "SON65P300X300X100-9N" H 3050 4850 50  0001 L CNN
+F 3 "http://www.ti.com/lit/gpn/TPS2556" H 3050 4750 50  0001 L CNN
+F 4 "Precision Adjustable Current-Limited Power-Distribution Switches  " H 3050 4650 50  0001 L CNN "Description"
+F 5 "" H 3050 4550 50  0001 L CNN "Height"
+F 6 "Texas Instruments" H 3050 4450 50  0001 L CNN "Manufacturer_Name"
+F 7 "TPS2556DRBR" H 3050 4350 50  0001 L CNN "Manufacturer_Part_Number"
+F 8 "595-TPS2556DRBR" H 3050 4250 50  0001 L CNN "Mouser Part Number"
+F 9 "https://www.mouser.co.uk/ProductDetail/Texas-Instruments/TPS2556DRBR?qs=PhbdE%2FyVlIdLuE1sx6iVjw%3D%3D" H 3050 4150 50  0001 L CNN "Mouser Price/Stock"
+F 10 "TPS2556DRBR" H 3050 4050 50  0001 L CNN "Arrow Part Number"
+F 11 "https://www.arrow.com/en/products/tps2556drbr/texas-instruments" H 3050 3950 50  0001 L CNN "Arrow Price/Stock"
+	1    2000 4750
+	1    0    0    -1
+$EndComp

Commit message: update microcontroller
Parts:
- removed IC?: MSP430F2274IYFFR, BGA49C40P7X7_333X349X62, symbol aalto-1-rescue:MSP430F2274IYFFR-MSP430F2274IYFFR
- added IC?: MSP430F2274IRHAT, QFN50P600X600X100-41N-D, symbol MSP430F2274IRHAT:MSP430F2274IRHAT
- IC?: symbol TPS2556DRBR:TPS2556DRBR -> aalto-1-rescue:TPS2556DRBR-TPS2556DRBR
Changed lines of the file:
@@
-$EndComp
-$Comp
-L aalto-1-rescue:MSP430F2274IYFFR-MSP430F2274IYFFR IC?
-U 1 1 603BEFA5
-P 6800 850
-F 0 "IC?" H 8350 1115 50  0000 C CNN
-F 1 "MSP430F2274IYFFR" H 8350 1024 50  0000 C CNN
-F 2 "BGA49C40P7X7_333X349X62" H 9750 950 50  0001 L CNN
-F 3 "http://www.ti.com/lit/gpn/msp430f2274" H 9750 850 50  0001 L CNN
-F 4 "16-bit Ultra-Low-Power Microcontroller, 32KB Flash, 1K RAM" H 9750 750 50  0001 L CNN "Description"
-F 5 "0.625" H 9750 650 50  0001 L CNN "Height"
-F 6 "Texas Instruments" H 9750 550 50  0001 L CNN "Manufacturer_Name"
-F 7 "MSP430F2274IYFFR" H 9750 450 50  0001 L CNN "Manufacturer_Part_Number"
-F 8 "595-MSP430F2274IYFFR" H 9750 350 50  0001 L CNN "Mouser Part Number"
-F 9 "https://www.mouser.com/Search/Refine.aspx?Keyword=595-MSP430F2274IYFFR" H 9750 250 50  0001 L CNN "Mouser Price/Stock"
-F 10 "MSP430F2274IYFFR" H 9750 150 50  0001 L CNN "Arrow Part Number"
-F 11 "https://www.arrow.com/en/products/msp430f2274iyffr/texas-instruments" H 9750 50  50  0001 L CNN "Arrow Price/Stock"
-	1    6800 850
-	1    0    0    -1
 $EndComp
 $Comp
@@
 $EndComp
 $Comp
-L TPS2556DRBR:TPS2556DRBR IC?
+L aalto-1-rescue:TPS2556DRBR-TPS2556DRBR IC?
 U 1 1 603C13A8
 P 2000 4750
@@
 	1    0    0    -1
 $EndComp
+$Comp
+L MSP430F2274IRHAT:MSP430F2274IRHAT IC?
+U 1 1 603BFCBF
+P 6850 1950
+F 0 "IC?" H 10694 1446 50  0000 L CNN
+F 1 "MSP430F2274IRHAT" H 10694 1355 50  0000 L CNN
+F 2 "QFN50P600X600X100-41N-D" H 10500 3050 50  0001 L CNN
+F 3 "http://www.ti.com/lit/ds/symlink/msp430f2274.pdf" H 10500 2950 50  0001 L CNN
+F 4 "MSP430F2274IRHAT, 16 bit MSP430 Microcontroller 16MHz 32kb Flash, 1kb RAM, I2C LIN SPI 40-Pin VQFN" H 10500 2850 50  0001 L CNN "Description"
+F 5 "1" H 10500 2750 50  0001 L CNN "Height"
+F 6 "Texas Instruments" H 10500 2650 50  0001 L CNN "Manufacturer_Name"
+F 7 "MSP430F2274IRHAT" H 10500 2550 50  0001 L CNN "Manufacturer_Part_Number"
+F 8 "595-MSP430F2274IRHAT" H 10500 2450 50  0001 L CNN "Mouser Part Number"
+F 9 "https://www.mouser.com/Search/Refine.aspx?Keyword=595-MSP430F2274IRHAT" H 10500 2350 50  0001 L CNN "Mouser Price/Stock"
+F 10 "MSP430F2274IRHAT" H 10500 2250 50  0001 L CNN "Arrow Part Number"
+F 11 "https://www.arrow.com/en/products/msp430f2274irhat/texas-instruments" H 10500 2150 50  0001 L CNN "Arrow Price/Stock"
+	1    6850 1950
+	1    0    0    -1
+$EndComp

Commit message: Just opened Kathryn's changes
I think it added cache files to the rescue folder so just uploading that as the "change"
Parts:
- IC?: symbol MSP430F2274IRHAT:MSP430F2274IRHAT -> aalto-1-rescue:MSP430F2274IRHAT-MSP430F2274IRHAT
Changed lines of the file:
@@
 $EndComp
 $Comp
-L MSP430F2274IRHAT:MSP430F2274IRHAT IC?
+L aalto-1-rescue:MSP430F2274IRHAT-MSP430F2274IRHAT IC?
 U 1 1 603BFCBF
 P 6850 1950

Commit message: add PA
Parts:
- added U?: RF5602, symbol aalto-1-rescue:RF5602
Changed lines of the file:
@@
+	1    0    0    -1
+$EndComp
+$Comp
+L aalto-1-rescue:RF5602 U?
+U 1 1 603F2812
+P 5100 1900
+F 0 "U?" H 5050 2715 50  0000 C CNN
+F 1 "RF5602" H 5050 2624 50  0000 C CNN
+F 2 "" H 5350 1200 50  0001 C CNN
+F 3 "" H 5350 1200 50  0001 C CNN
+	1    5100 1900
 	1    0    0    -1
 $EndComp
