File: aalto-1/aalto-1.sch (KiCad schematic (older format))
At the start: 5 parts

Commit message: labeling
Changed lines of the file:
@@
 	1    0    0    -1
 $EndComp
+Text Label 5300 1200 0    50   ~ 0
+PowerAmplifier
+Text Label 9800 800  0    50   ~ 0
+Microcontroller
+Text Label 2950 4550 0    50   ~ 0
+PowerSwitch
+Text Label 6150 3400 0    50   ~ 0
+RFTransciever
 $EndSCHEMATC
