File: aalto-1/PA + PS.sch (KiCad schematic (older format))
At the start: 0 parts

Commit message: Finished schematic rough draft
Parts:
- added C?: 330pF, symbol Device:C
- added C?: 1nF, symbol Device:C
- added C?: 4.7pF, symbol Device:C
- added IC?: RFPA5200-RFPA5200, RFPA5200, symbol aalto-1-rescue:RFPA5200-RFPA5200
- added L?: 1.8nH, symbol Device:L
- added R? (x4): R, symbol Device:R
Connections:
- new net: IC?.9 (VREG), R?.2
- new net: C?.1, L?.1, R?.1
- new net GND: C?.2, C?.2, C?.2, IC?.2 (GND_1), IC?.4 (NC/_GND), IC?.7 (GND_2), IC?.8 (GND_3), R?.2
- new net PDETECT_RF5200: C?.1, IC?.5 (PDET)
- new net RFOUT: IC?.6 (RFOUT)
- new net RF_IN: IC?.1 (RFIN)
- new net VCC_PA: R?.1, R?.2
- new net VCC_RF5200: IC?.3 (VCC), L?.2
- new net VREG: C?.1, IC?.10 (PA_EN), R?.1, R?.1, R?.2
