File: aalto-1/Microcontroller + Bus.sch (KiCad schematic (older format))
At the start: 1 part

Commit message: update 3/14
Parts:
- added C? (x3): C, symbol Device:C
- added IC?: TPS2556DRBR-TPS2556DRBR, SON65P300X300X100-9N, symbol aalto-1-rescue:TPS2556DRBR-TPS2556DRBR
- added R?: R, symbol Device:R
Connections:
- net labels added: CLK_OBC, FAULT, GDO0_CC2500, GDO2_CC2500, GND-power, PDEDECT_RF5602, PDOWN, SIMO_CC2500, SOMI_CC2500, SPY_BY_WIRE_RST, VCC
- wire segments 12 -> 51
Other:
- moved on the sheet: IC?

Commit message: Finished schematic rough draft
Parts:
- added C?: 0.1μF, symbol Device:C
- added C?: 0.004μF, symbol Device:C
- added J? (x2): Conn_2Rows-53Pins, symbol Connector_Generic:Conn_2Rows-53Pins
- added R?: R, symbol Device:R
- C? (x2): value C -> 0.1μF
- C?: value C -> 0.004μF
- R?: value R -> 174kΩ
Connections:
- net FAULT: now also IC?.33 (P1.4/SMCLK/TCK), J?.25 (Pin_25)
- net GND: now also C?.2, C?.2, J?.14 (Pin_14), J?.25 (Pin_25), J?.30 (Pin_30), J?.32 (Pin_32), J?.33 (Pin_33), J?.34 (Pin_34), J?.39 (Pin_39), J?.40 (Pin_40), J?.5 (Pin_5), J?.6 (Pin_6), J?.8 (Pin_8)
- net PDOWN: now also IC?.32 (P1.3/TA2)
- net SPY_BY_WIRE_RST: now also J?.20 (Pin_20)
- net CLK_CC2500: now reaches IC?.12 (P3.3/UCB0CLK/UCA0STE)
- net VCC3.3: now reaches IC?.14 (AVCC)
- net PROG_RX: now reaches IC?.24 (P3.5/UCA0RXD/UCA0SOMI)
- net PROG_RX: now also J?.15 (Pin_15)
- net CSN_CC2500: now reaches IC?.30 (P1.1/TA0)
- net SPY_BY_WIRE_TEST: now reaches IC?.37 (TEST/SBWTCK)
- net SPY_BY_WIRE_TEST: now also J?.19 (Pin_19)
- new net 3.3GPS: J?.28 (Pin_28), R?.1
- new net GPS_BOOT_SELECT: J?.19 (Pin_19)
- new net GPS_ENABLE: J?.20 (Pin_20)
- new net GPS_PPS: J?.13 (Pin_13)
- new net GPS_RESET: J?.14 (Pin_14)
- new net GPS_RX: J?.12 (Pin_12)
- new net GPS_TX: J?.11 (Pin_11)
- new net MOSI_OBC: J?.17 (Pin_17)
- new net OBC_CSN: J?.21 (Pin_21)
- new net SBAND_CLK+: J?.9 (Pin_9)
- new net SBAND_CLK-: J?.10 (Pin_10)
- new net SBAND_MOSI+: J?.11 (Pin_11)
- new net SBAND_MOSI-: J?.12 (Pin_12)
- new net VCC_3.3: C?.1, C?.1, J?.27 (Pin_27), R?.2

Commit message: Labeling schematics
Connections:
- net +3V3 is gone; now on net VCC3.3: IC?.38 (DVCC), IC?.39 (DVCC_1)
- net VCC_3.3 is gone; now on net VCC3.3: C?.1, C?.1, J?.27 (Pin_27), R?.2
- net VCC_PA: now reaches C?.1, C?.1, IC?.6 (OUT_2), IC?.7 (OUT)
- net PDEDECT_RF5602 renamed PDETECT_RF5200
Changed lines of the file:
@@
 Wire Wire Line
 	7500 2250 5850 2250
-$Comp
-L aalto-1-rescue:+3.3V-power #PWR?
-U 1 1 604880D4
-P 7750 2150
-AR Path="/604880D4" Ref="#PWR?"  Part="1"
-AR Path="/6048217D/604880D4" Ref="#PWR?"  Part="1"
-F 0 "#PWR?" H 7750 2000 50  0001 C CNN
-F 1 "+3.3V" H 7765 2323 50  0000 C CNN
-F 2 "" H 7750 2150 50  0001 C CNN
-F 3 "" H 7750 2150 50  0001 C CNN
-	1    7750 2150
-	1    0    0    -1
-$EndComp
 Wire Wire Line
 	7700 2250 7750 2250
@@
 Connection ~ 3700 2050
 Wire Wire Line
-	3700 2050 4350 2050
+	3700 2050 4250 2050
 $Comp
 L aalto-1-rescue:GND-power #PWR?
@@
 	1    0    0    -1
 $EndComp
-Text Label 5300 3650 0    50   ~ 0
-GDO2_CC2500
-Wire Wire Line
-	6100 3650 5300 3650
-Text Label 5300 3750 0    50   ~ 0
-GDO0_CC2500
-Wire Wire Line
-	6100 3750 5300 3750
-Text Label 5300 3950 0    50   ~ 0
-SPY_BY_WIRE_RST
-Wire Wire Line
-	6100 3950 5300 3950
-Text Label 5300 4050 0    50   ~ 0
-PDEDECT_RF5602
-Wire Wire Line
-	6100 4050 5300 4050
-Text Label 5300 4350 0    50   ~ 0
-CLK_OBC
-Wire Wire Line
-	6100 4350 5300 4350
-Text Label 5300 4450 0    50   ~ 0
-SIMO_CC2500
 Wire Wire Line
 	6100 4450 5300 4450
-Text Label 7500 6200 3    50   ~ 0
-SOMI_CC2500
 Wire Wire Line
 	7500 5950 7500 6200
-Text Label 7600 6200 3    50   ~ 0
-CLK_CC2500
-Wire Wire Line
-	7600 6450 7600 5950
-Text Label 7800 6250 3    50   ~ 0
-VCC3.3
-Wire Wire Line
-	7800 6250 7800 5950
-Text Label 10400 4150 2    50   ~ 0
-PROG_RX
 Wire Wire Line
 	9900 4150 10400 4150
-Text Label 10550 3550 2    50   ~ 0
-CSN_CC2500
 Wire Wire Line
 	9900 3550 10550 3550
-Text Label 8400 1950 3    50   ~ 0
-PDOWN
 Wire Wire Line
 	8400 2250 8400 1950
-Text Label 8300 1950 3    50   ~ 0
-FAULT
 Wire Wire Line
 	8300 1950 8300 2250
-Text Label 7900 1200 3    50   ~ 0
-SPY_BY_WIRE_TEST
 Wire Wire Line
 	7900 1200 7900 2250
@@
 Wire Wire Line
 	2900 6050 2900 5700
-Text Label 1600 5700 2    50   ~ 0
-VCC_3.3
 Wire Wire Line
 	1600 5700 1800 5700
@@
 Wire Wire Line
 	3900 4950 4100 4950
+Text GLabel 4950 3650 0    50   Input ~ 0
+GDO2_CC2500
+Text GLabel 4950 3950 0    50   Input ~ 0
+SPY_BY_WIRE_RST
+Text GLabel 5700 4050 0    50   Input ~ 0
+PDETECT_RF5200
+Text GLabel 5700 4350 0    50   Input ~ 0
+CLK_OBC
+Text GLabel 5300 4450 0    50   Input ~ 0
+SIMO_CC2500
+Text GLabel 7500 6200 0    50   Input ~ 0
+SOMI_CC2500
+Text GLabel 7550 6350 0    50   Input ~ 0
+CLK_CC2500
+Text GLabel 7750 6450 0    50   Input ~ 0
+VCC3.3
+Text GLabel 10550 3550 2    50   Input ~ 0
+CSN_CC2500
+Text GLabel 5700 3750 0    50   Input ~ 0
+GDO0_CC2500
+Wire Wire Line
+	6100 4350 5700 4350
+Wire Wire Line
+	6100 4050 5700 4050
+Wire Wire Line
+	4950 3950 6100 3950
+Wire Wire Line
+	5700 3750 6100 3750
+Wire Wire Line
+	4950 3650 6100 3650
+Wire Wire Line
+	7750 6450 7800 6450
+Wire Wire Line
+	7800 5950 7800 6450
+Wire Wire Line
+	7550 6350 7600 6350
+Wire Wire Line
+	7600 6350 7600 5950
+Text Label 8400 1950 0    50   ~ 0
+PDOWN
+Text Label 8300 1950 2    50   ~ 0
+FAULT
+Text Label 7900 1200 2    50   ~ 0
+SPY_BY_WIRE_TEST
+Text Label 10400 4150 0    50   ~ 0
+PROG_RX
+Text GLabel 7750 2150 0    50   Input ~ 0
+VCC3.3
+Text GLabel 900  5700 0    50   Input ~ 0
+VCC3.3
+Text GLabel 4250 1850 0    50   Input ~ 0
+VCC_PA
+Wire Wire Line
+	4250 1850 4250 2050
+Connection ~ 4250 2050
+Wire Wire Line
+	4250 2050 4350 2050
 $EndSCHEMATC

Commit message: starting pcb layout
Parts:
- gave numbers to parts that had none: 11
Connections:
- net OBC_CSN: now also IC2.31 (P1.2/TA1)
- net SBAND_CLK-: no longer names the net of J1.10 (Pin_10)
- net SBAND_MOSI-: no longer names the net of J1.12 (Pin_12)
Changed lines of the file:
@@
 	7750 2250 7800 2250
 $Comp
-L aalto-1-rescue:TPS2556DRBR-TPS2556DRBR IC?
+L aalto-1-rescue:TPS2556DRBR-TPS2556DRBR IC1
 U 1 1 604E64C5
 P 2300 1950
-F 0 "IC?" H 2900 2215 50  0000 C CNN
+F 0 "IC1" H 2900 2215 50  0000 C CNN
 F 1 "TPS2556DRBR-TPS2556DRBR" H 2900 2124 50  0000 C CNN
 F 2 "SON65P300X300X100-9N" H 3350 2050 50  0001 L CNN
@@
 $EndComp
 $Comp
-L Device:R R?
+L Device:R R1
 U 1 1 604E77DC
 P 2000 2750
-F 0 "R?" H 2070 2796 50  0000 L CNN
+F 0 "R1" H 2070 2796 50  0000 L CNN
 F 1 "174kΩ" H 2070 2705 50  0000 L CNN
 F 2 "" V 1930 2750 50  0001 C CNN
@@
 $EndComp
 $Comp
-L aalto-1-rescue:GND-power #PWR?
+L aalto-1-rescue:GND-power #PWR03
 U 1 1 604E86B4
 P 1450 1550
-F 0 "#PWR?" H 1450 1300 50  0001 C CNN
+F 0 "#PWR03" H 1450 1300 50  0001 C CNN
 F 1 "GND-power" H 1455 1377 50  0000 C CNN
 F 2 "" H 1450 1550 50  0001 C CNN
@@
 VCC
 $Comp
-L aalto-1-rescue:GND-power #PWR?
+L aalto-1-rescue:GND-power #PWR04
 U 1 1 604F0802
 P 1500 2600
-F 0 "#PWR?" H 1500 2350 50  0001 C CNN
+F 0 "#PWR04" H 1500 2350 50  0001 C CNN
 F 1 "GND-power" H 1505 2427 50  0000 C CNN
 F 2 "" H 1500 2600 50  0001 C CNN
@@
 	1750 1300 1750 2150
 $Comp
-L Device:C C?
+L Device:C C3
 U 1 1 604F6B4D
 P 1500 2300
-F 0 "C?" H 1615 2346 50  0000 L CNN
+F 0 "C3" H 1615 2346 50  0000 L CNN
 F 1 "0.1μF" H 1615 2255 50  0000 L CNN
 F 2 "" H 1538 2150 50  0001 C CNN
@@
 	2150 2150 1750 2150
 $Comp
-L Device:C C?
+L Device:C C5
 U 1 1 604F7B33
 P 4800 2600
-F 0 "C?" H 4915 2646 50  0000 L CNN
+F 0 "C5" H 4915 2646 50  0000 L CNN
 F 1 "0.004μF" H 4915 2555 50  0000 L CNN
 F 2 "" H 4838 2450 50  0001 C CNN
@@
 $EndComp
 $Comp
-L Device:C C?
+L Device:C C4
 U 1 1 604F8F6E
 P 4350 2600
-F 0 "C?" H 4465 2646 50  0000 L CNN
+F 0 "C4" H 4465 2646 50  0000 L CNN
 F 1 "0.1μF" H 4465 2555 50  0000 L CNN
 F 2 "" H 4388 2450 50  0001 C CNN
@@
 $EndComp
 $Comp
-L aalto-1-rescue:GND-power #PWR?
+L aalto-1-rescue:GND-power #PWR010
 U 1 1 604F9393
 P 4800 2950
-F 0 "#PWR?" H 4800 2700 50  0001 C CNN
+F 0 "#PWR010" H 4800 2700 50  0001 C CNN
 F 1 "GND-power" H 4805 2777 50  0000 C CNN
 F 2 "" H 4800 2950 50  0001 C CNN
@@
 $EndComp
 $Comp
-L aalto-1-rescue:GND-power #PWR?
+L aalto-1-rescue:GND-power #PWR09
 U 1 1 604F95F2
 P 4350 2950
-F 0 "#PWR?" H 4350 2700 50  0001 C CNN
+F 0 "#PWR09" H 4350 2700 50  0001 C CNN
 F 1 "GND-power" H 4355 2777 50  0000 C CNN
 F 2 "" H 4350 2950 50  0001 C CNN
@@
 	3700 2050 4250 2050
 $Comp
-L aalto-1-rescue:GND-power #PWR?
+L aalto-1-rescue:GND-power #PWR08
 U 1 1 604FC070
 P 3700 2550
-F 0 "#PWR?" H 3700 2300 50  0001 C CNN
+F 0 "#PWR08" H 3700 2300 50  0001 C CNN
 F 1 "GND-power" H 3705 2377 50  0000 C CNN
 F 2 "" H 3700 2550 50  0001 C CNN
@@
 	6100 3550 5850 3550
 $Comp
-L aalto-1-rescue:GND-power #PWR?
+L aalto-1-rescue:GND-power #PWR012
 U 1 1 604861CC
 P 5850 6100
-F 0 "#PWR?" H 5850 5850 50  0001 C CNN
+F 0 "#PWR012" H 5850 5850 50  0001 C CNN
 F 1 "GND" H 5855 5927 50  0000 C CNN
 F 2 "" H 5850 6100 50  0001 C CNN
@@
 $EndComp
 $Comp
-L aalto-1-rescue:MSP430F2274IRHAT-MSP430F2274IRHAT IC?
+L aalto-1-rescue:MSP430F2274IRHAT-MSP430F2274IRHAT IC2
 U 1 1 60482A2A
 P 6100 3550
-F 0 "IC?" H 7050 3700 50  0000 L CNN
+F 0 "IC2" H 7050 3700 50  0000 L CNN
 F 1 "MSP430F2274IRHAT-MSP430F2274IRHAT" H 7250 3700 50  0000 L CNN
 F 2 "QFN50P600X600X100-41N-D" H 9750 4650 50  0001 L CNN
@@
 	7900 1200 7900 2250
 $Comp
-L Connector_Generic:Conn_2Rows-53Pins J?
+L Connector_Generic:Conn_2Rows-53Pins J1
 U 1 1 6059B65A
 P 2000 5700
-F 0 "J?" H 2050 7217 50  0000 C CNN
+F 0 "J1" H 2050 7217 50  0000 C CNN
 F 1 "Conn_2Rows-53Pins" H 2050 7126 50  0000 C CNN
 F 2 "" H 2000 5700 50  0001 C CNN
@@
 $EndComp
 $Comp
-L Connector_Generic:Conn_2Rows-53Pins J?
+L Connector_Generic:Conn_2Rows-53Pins J2
 U 1 1 605A3F15
 P 4300 5750
-F 0 "J?" H 4350 7267 50  0000 C CNN
+F 0 "J2" H 4350 7267 50  0000 C CNN
 F 1 "Conn_2Rows-53Pins" H 4350 7176 50  0000 C CNN
 F 2 "" H 4300 5750 50  0001 C CNN
@@
 	1600 5600 1800 5600
 $Comp
-L power:GND #PWR?
+L power:GND #PWR06
 U 1 1 605B744F
 P 2950 5000
-F 0 "#PWR?" H 2950 4750 50  0001 C CNN
+F 0 "#PWR06" H 2950 4750 50  0001 C CNN
 F 1 "GND" H 2955 4827 50  0000 C CNN
 F 2 "" H 2950 5000 50  0001 C CNN
@@
 Wire Wire Line
 	2300 5000 2950 5000
-Text Label 2800 4800 2    50   ~ 0
-SBAND_CLK-
-Text Label 2850 4900 2    50   ~ 0
-SBAND_MOSI-
-Wire Wire Line
-	2850 4900 2300 4900
-Wire Wire Line
-	2800 4800 2300 4800
 Text Label 3000 5300 2    50   ~ 0
 SPY_BY_WIRE_RST
@@
 3.3GPS
 $Comp
-L power:GND #PWR?
+L power:GND #PWR05
 U 1 1 605D0A4B
 P 2600 5950
-F 0 "#PWR?" H 2600 5700 50  0001 C CNN
+F 0 "#PWR05" H 2600 5700 50  0001 C CNN
 F 1 "GND" H 2605 5777 50  0000 C CNN
 F 2 "" H 2600 5950 50  0001 C CNN
@@
 	2600 5800 2600 5900
 $Comp
-L Device:R R?
+L Device:R R2
 U 1 1 605DC196
 P 2900 6200
-F 0 "R?" H 2970 6246 50  0000 L CNN
+F 0 "R2" H 2970 6246 50  0000 L CNN
 F 1 "R" H 2970 6155 50  0000 L CNN
 F 2 "" V 2830 6200 50  0001 C CNN
@@
 	2300 5700 2900 5700
 $Comp
-L Device:C C?
+L Device:C C1
 U 1 1 605E5108
 P 700 6400
-F 0 "C?" H 815 6446 50  0000 L CNN
+F 0 "C1" H 815 6446 50  0000 L CNN
 F 1 "0.1μF" H 815 6355 50  0000 L CNN
 F 2 "" H 738 6250 50  0001 C CNN
@@
 $EndComp
 $Comp
-L Device:C C?
+L Device:C C2
 U 1 1 605E5A2E
 P 1150 6400
-F 0 "C?" H 1265 6446 50  0000 L CNN
+F 0 "C2" H 1265 6446 50  0000 L CNN
 F 1 "0.004μF" H 1265 6355 50  0000 L CNN
 F 2 "" H 1188 6250 50  0001 C CNN
@@
 Connection ~ 1600 5700
 $Comp
-L power:GND #PWR?
+L power:GND #PWR01
 U 1 1 605EA99D
 P 700 6550
-F 0 "#PWR?" H 700 6300 50  0001 C CNN
+F 0 "#PWR01" H 700 6300 50  0001 C CNN
 F 1 "GND" H 705 6377 50  0000 C CNN
 F 2 "" H 700 6550 50  0001 C CNN
@@
 $EndComp
 $Comp
-L power:GND #PWR?
+L power:GND #PWR02
 U 1 1 605EB0FD
 P 1150 6550
-F 0 "#PWR?" H 1150 6300 50  0001 C CNN
+F 0 "#PWR02" H 1150 6300 50  0001 C CNN
 F 1 "GND" H 1155 6377 50  0000 C CNN
 F 2 "" H 1150 6550 50  0001 C CNN
@@
 	900  5700 1600 5700
 $Comp
-L power:GND #PWR?
+L power:GND #PWR07
 U 1 1 605F9A31
 P 3400 6350
-F 0 "#PWR?" H 3400 6100 50  0001 C CNN
+F 0 "#PWR07" H 3400 6100 50  0001 C CNN
 F 1 "GND" H 3405 6177 50  0000 C CNN
 F 2 "" H 3400 6350 50  0001 C CNN
@@
 Connection ~ 3400 5650
 $Comp
-L power:GND #PWR?
+L power:GND #PWR011
 U 1 1 606037E3
 P 5350 6350
-F 0 "#PWR?" H 5350 6100 50  0001 C CNN
+F 0 "#PWR011" H 5350 6100 50  0001 C CNN
 F 1 "GND" H 5355 6177 50  0000 C CNN
 F 2 "" H 5350 6350 50  0001 C CNN
@@
 Text GLabel 4950 3650 0    50   Input ~ 0
 GDO2_CC2500
-Text GLabel 4950 3950 0    50   Input ~ 0
-SPY_BY_WIRE_RST
 Text GLabel 5700 4050 0    50   Input ~ 0
 PDETECT_RF5200
-Text GLabel 5700 4350 0    50   Input ~ 0
-CLK_OBC
 Text GLabel 5300 4450 0    50   Input ~ 0
 SIMO_CC2500
@@
 Wire Wire Line
 	4250 2050 4350 2050
+Text Label 8500 2100 0    50   ~ 0
+OBC_CSN
+Wire Wire Line
+	8500 2100 8500 2250
+Text Label 4950 3950 2    50   ~ 0
+SPY_BY_WIRE_RST
+Text Label 5700 4350 2    50   ~ 0
+CLK_OBC
 $EndSCHEMATC

Commit message: footprint libraries
Parts:
- IC2: footprint QFN50P600X600X100-41N-D -> MSP430F2274IRHAT:QFN50P600X600X100-41N-D
- J1, J2: symbol Connector_Generic:Conn_2Rows-53Pins -> aalto-1-rescue:Conn_2Rows-53Pins-Connector_Generic
Changed lines of the file:
@@
 F 0 "IC2" H 7050 3700 50  0000 L CNN
 F 1 "MSP430F2274IRHAT-MSP430F2274IRHAT" H 7250 3700 50  0000 L CNN
-F 2 "QFN50P600X600X100-41N-D" H 9750 4650 50  0001 L CNN
+F 2 "MSP430F2274IRHAT:QFN50P600X600X100-41N-D" H 9750 4650 50  0001 L CNN
 F 3 "http://www.ti.com/lit/ds/symlink/msp430f2274.pdf" H 9750 4550 50  0001 L CNN
 F 4 "MSP430F2274IRHAT, 16 bit MSP430 Microcontroller 16MHz 32kb Flash, 1kb RAM, I2C LIN SPI 40-Pin VQFN" H 9750 4450 50  0001 L CNN "Description"
@@
 	7900 1200 7900 2250
 $Comp
-L Connector_Generic:Conn_2Rows-53Pins J1
+L aalto-1-rescue:Conn_2Rows-53Pins-Connector_Generic J1
 U 1 1 6059B65A
 P 2000 5700
@@
 $EndComp
 $Comp
-L Connector_Generic:Conn_2Rows-53Pins J2
+L aalto-1-rescue:Conn_2Rows-53Pins-Connector_Generic J2
 U 1 1 605A3F15
 P 4300 5750
@@
 	1600 5600 1800 5600
 $Comp
-L power:GND #PWR06
+L aalto-1-rescue:GND-power #PWR06
 U 1 1 605B744F
 P 2950 5000
@@
 3.3GPS
 $Comp
-L power:GND #PWR05
+L aalto-1-rescue:GND-power #PWR05
 U 1 1 605D0A4B
 P 2600 5950
@@
 Connection ~ 1600 5700
 $Comp
-L power:GND #PWR01
+L aalto-1-rescue:GND-power #PWR01
 U 1 1 605EA99D
 P 700 6550
@@
 $EndComp
 $Comp
-L power:GND #PWR02
+L aalto-1-rescue:GND-power #PWR02
 U 1 1 605EB0FD
 P 1150 6550
@@
 	900  5700 1600 5700
 $Comp
-L power:GND #PWR07
+L aalto-1-rescue:GND-power #PWR07
 U 1 1 605F9A31
 P 3400 6350
@@
 Connection ~ 3400 5650
 $Comp
-L power:GND #PWR011
+L aalto-1-rescue:GND-power #PWR011
 U 1 1 606037E3
 P 5350 6350

Commit message: Fall 2021
Parts:
- C1, C2, C3, C4, C5: footprint (none) -> Capacitor_SMD:C_0805_2012Metric
- R1, R2: footprint (none) -> Resistor_SMD:R_0805_2012Metric
Connections:
- net SBAND_CLK-: now reaches J1.10 (Pin_10)
- net SBAND_MOSI-: now reaches J1.12 (Pin_12)
Changed lines of the file:
@@
 F 0 "R1" H 2070 2796 50  0000 L CNN
 F 1 "174kΩ" H 2070 2705 50  0000 L CNN
-F 2 "" V 1930 2750 50  0001 C CNN
+F 2 "Resistor_SMD:R_0805_2012Metric" V 1930 2750 50  0001 C CNN
 F 3 "~" H 2000 2750 50  0001 C CNN
 	1    2000 2750
@@
 F 0 "C3" H 1615 2346 50  0000 L CNN
 F 1 "0.1μF" H 1615 2255 50  0000 L CNN
-F 2 "" H 1538 2150 50  0001 C CNN
+F 2 "Capacitor_SMD:C_0805_2012Metric" H 1538 2150 50  0001 C CNN
 F 3 "~" H 1500 2300 50  0001 C CNN
 	1    1500 2300
@@
 F 0 "C5" H 4915 2646 50  0000 L CNN
 F 1 "0.004μF" H 4915 2555 50  0000 L CNN
-F 2 "" H 4838 2450 50  0001 C CNN
+F 2 "Capacitor_SMD:C_0805_2012Metric" H 4838 2450 50  0001 C CNN
 F 3 "~" H 4800 2600 50  0001 C CNN
 	1    4800 2600
@@
 F 0 "C4" H 4465 2646 50  0000 L CNN
 F 1 "0.1μF" H 4465 2555 50  0000 L CNN
-F 2 "" H 4388 2450 50  0001 C CNN
+F 2 "Capacitor_SMD:C_0805_2012Metric" H 4388 2450 50  0001 C CNN
 F 3 "~" H 4350 2600 50  0001 C CNN
 	1    4350 2600
@@
 	7900 1200 7900 2250
 $Comp
-L aalto-1-rescue:Conn_2Rows-53Pins-Connector_Generic J1
-U 1 1 6059B65A
-P 2000 5700
-F 0 "J1" H 2050 7217 50  0000 C CNN
-F 1 "Conn_2Rows-53Pins" H 2050 7126 50  0000 C CNN
-F 2 "" H 2000 5700 50  0001 C CNN
-F 3 "~" H 2000 5700 50  0001 C CNN
-	1    2000 5700
-	1    0    0    -1
-$EndComp
-$Comp
 L aalto-1-rescue:Conn_2Rows-53Pins-Connector_Generic J2
 U 1 1 605A3F15
@@
 	2950 4700 2950 5000
 Connection ~ 2950 5000
-Wire Wire Line
-	2300 4700 2950 4700
-Wire Wire Line
-	2300 5000 2950 5000
 Text Label 3000 5300 2    50   ~ 0
 SPY_BY_WIRE_RST
-Wire Wire Line
-	3000 5300 2300 5300
 Text Label 3200 5700 2    50   ~ 0
 3.3GPS
@@
 Wire Wire Line
 	2600 5950 2600 5900
-Wire Wire Line
-	2300 5900 2600 5900
 Connection ~ 2600 5900
-Wire Wire Line
-	2300 5800 2600 5800
 Wire Wire Line
 	2600 5800 2600 5900
@@
 F 0 "R2" H 2970 6246 50  0000 L CNN
 F 1 "R" H 2970 6155 50  0000 L CNN
-F 2 "" V 2830 6200 50  0001 C CNN
+F 2 "Resistor_SMD:R_0805_2012Metric" V 2830 6200 50  0001 C CNN
 F 3 "~" H 2900 6200 50  0001 C CNN
 	1    2900 6200
@@
 Wire Wire Line
 	2900 5700 3200 5700
-Wire Wire Line
-	2300 5700 2900 5700
 $Comp
 L Device:C C1
@@
 F 0 "C1" H 815 6446 50  0000 L CNN
 F 1 "0.1μF" H 815 6355 50  0000 L CNN
-F 2 "" H 738 6250 50  0001 C CNN
+F 2 "Capacitor_SMD:C_0805_2012Metric" H 738 6250 50  0001 C CNN
 F 3 "~" H 700 6400 50  0001 C CNN
 	1    700  6400
@@
 F 0 "C2" H 1265 6446 50  0000 L CNN
 F 1 "0.004μF" H 1265 6355 50  0000 L CNN
-F 2 "" H 1188 6250 50  0001 C CNN
+F 2 "Capacitor_SMD:C_0805_2012Metric" H 1188 6250 50  0001 C CNN
 F 3 "~" H 1150 6400 50  0001 C CNN
 	1    1150 6400
@@
 Text Label 5700 4350 2    50   ~ 0
 CLK_OBC
+Wire Wire Line
+	2300 5900 2600 5900
+Wire Wire Line
+	2300 5800 2600 5800
+Wire Wire Line
+	2300 5700 2900 5700
+Wire Wire Line
+	3000 5300 2300 5300
+Wire Wire Line
+	2300 5000 2950 5000
+Wire Wire Line
+	2300 4700 2950 4700
+Text Label 2450 4900 0    50   ~ 0
+SBAND_MOSI-
+$Comp
+L aalto-1-rescue:Conn_2Rows-53Pins-Connector_Generic J1
+U 1 1 6059B65A
+P 2000 5700
+F 0 "J1" H 2050 7217 50  0000 C CNN
+F 1 "Conn_2Rows-53Pins" H 2050 7126 50  0000 C CNN
+F 2 "" H 2000 5700 50  0001 C CNN
+F 3 "~" H 2000 5700 50  0001 C CNN
+	1    2000 5700
+	1    0    0    -1
+$EndComp
+Text Label 2450 4800 0    50   ~ 0
+SBAND_CLK-
+Wire Wire Line
+	2300 4800 2450 4800
+Wire Wire Line
+	2300 4900 2450 4900
 $EndSCHEMATC
